File: OSHEGrowbotBotPDB/OSHEGrowbotBotPDB.kicad_pcb (KiCad board)
At the start: 2 copper layers, 50 x 80 mm, 12 parts, among them J1 Battery Connector, J2 5V Regulator, J3 Voltage Sense, J4 5V Rail, J5 Ground Rail, J6 Motor Power

Commit message: Final draft, time for verification
Parts:
- removed J6: Motor Power, OSHEGrowbotBotPDB:pxc_1017521_00_TDPT-4-2-SP-6-35-ZB
- J1: value Battery Connector -> Battery; footprint OSHEGrowbotBotPDB:pxc_1017521_00_TDPT-4-2-SP-6-35-ZB -> OSHEGrowbotBotPDB:pxc_1984963_04_PTSA-1-5-2-3-5-F
- moved J2 11.9 mm to (99.8, 53.3)
- moved R1 7.57 mm to (111.1, 83.2), turned to 270 degrees
- moved R2 6.57 mm to (117.1, 90.8), turned to 90 degrees
- moved J3 4.89 mm to (111.7, 118.1)
- moved J1 0.10 mm to (92.7, 96.1)
Routing:
- net Net-(J1-Pad2): track 0.00 -> 96.8 mm
- net Net-(J1-Pad1): track 0.00 -> 61.0 mm
- net Net-(J2-Pad4): track 0.00 -> 58.9 mm
- net Net-(J2-Pad3): track 0.00 -> 58.3 mm
- net Net-(J3-Pad1): track 0.00 -> 41.5 mm
Other:
- net class Default: clearance 0.2 -> 0.5; trace_width 0.25 -> 2.5
- net class Power added: clearance 0.5, trace_width 2.5, via_dia 0.8, via_drill 0.4
- net class Vbat removed
- rule trace_clearance: 0.2 -> 0.5
